File: LNA_Gain_Ctrl.sch (KiCad schematic (older format))
At the start: 10 parts, among them U2 TLV73311PDBVT, U3 MAX5387LAUD+T

Commit message: Assigned footprint for dimension checking
Parts:
- R13, R14, R15, R16, R17, R18, R19, R20: footprint Resistors_SMD:R_0603 -> Resistors_SMD:R_0603_HandSoldering
Changed lines of the file:
@@
 LIBS:contrib
 LIBS:valves
+LIBS:zeabus
 LIBS:ftdi
 LIBS:zeabus-elec-hydrophone-frontend-cache
@@
 $EndComp
 $Comp
-L GNDA #PWR30
+L GNDA #PWR028
 U 1 1 599B078D
 P 7350 2300
-F 0 "#PWR30" H 7350 2050 50  0001 C CNN
+F 0 "#PWR028" H 7350 2050 50  0001 C CNN
 F 1 "GNDA" H 7350 2150 50  0000 C CNN
 F 2 "" H 7350 2300 50  0001 C CNN
@@
 $EndComp
 $Comp
-L +3.3VA #PWR31
+L +3.3VA #PWR029
 U 1 1 599B07B0
 P 8250 2050
-F 0 "#PWR31" H 8250 1900 50  0001 C CNN
+F 0 "#PWR029" H 8250 1900 50  0001 C CNN
 F 1 "+3.3VA" H 8250 2190 50  0000 C CNN
 F 2 "" H 8250 2050 50  0001 C CNN
@@
 	6600 3950 6550 3950
 $Comp
-L GNDA #PWR29
+L GNDA #PWR030
 U 1 1 599B08BC
 P 7000 4050
-F 0 "#PWR29" H 7000 3800 50  0001 C CNN
+F 0 "#PWR030" H 7000 3800 50  0001 C CNN
 F 1 "GNDA" H 7000 3900 50  0000 C CNN
 F 2 "" H 7000 4050 50  0001 C CNN
@@
 	5150 4150 5150 4450
 $Comp
-L GNDD #PWR27
+L GNDD #PWR031
 U 1 1 599B08F3
 P 5150 4450
-F 0 "#PWR27" H 5150 4200 50  0001 C CNN
+F 0 "#PWR031" H 5150 4200 50  0001 C CNN
 F 1 "GNDD" H 5150 4300 50  0000 C CNN
 F 2 "" H 5150 4450 50  0001 C CNN
@@
 $EndComp
 $Comp
-L +3.3V #PWR26
+L +3.3V #PWR032
 U 1 1 599B0916
 P 5150 3150
-F 0 "#PWR26" H 5150 3000 50  0001 C CNN
+F 0 "#PWR032" H 5150 3000 50  0001 C CNN
 F 1 "+3.3V" H 5150 3290 50  0000 C CNN
 F 2 "" H 5150 3150 50  0001 C CNN
@@
 F 0 "R18" V 4180 4200 50  0000 C CNN
 F 1 "10k" V 4100 4200 50  0000 C CNN
-F 2 "Resistors_SMD:R_0603" V 4030 4200 50  0001 C CNN
+F 2 "Resistors_SMD:R_0603_HandSoldering" V 4030 4200 50  0001 C CNN
 F 3 "" H 4100 4200 50  0001 C CNN
 	1    4100 4200
@@
 F 0 "R19" V 4380 4200 50  0000 C CNN
 F 1 "10k" V 4300 4200 50  0000 C CNN
-F 2 "Resistors_SMD:R_0603" V 4230 4200 50  0001 C CNN
+F 2 "Resistors_SMD:R_0603_HandSoldering" V 4230 4200 50  0001 C CNN
 F 3 "" H 4300 4200 50  0001 C CNN
 	1    4300 4200
@@
 F 0 "R20" V 4580 4200 50  0000 C CNN
 F 1 "10k" V 4500 4200 50  0000 C CNN
-F 2 "Resistors_SMD:R_0603" V 4430 4200 50  0001 C CNN
+F 2 "Resistors_SMD:R_0603_HandSoldering" V 4430 4200 50  0001 C CNN
 F 3 "" H 4500 4200 50  0001 C CNN
 	1    4500 4200
@@
 F 0 "R14" V 4180 3400 50  0000 C CNN
 F 1 "0" V 4100 3400 50  0000 C CNN
-F 2 "Resistors_SMD:R_0603" V 4030 3400 50  0001 C CNN
+F 2 "Resistors_SMD:R_0603_HandSoldering" V 4030 3400 50  0001 C CNN
 F 3 "" H 4100 3400 50  0001 C CNN
 	1    4100 3400
@@
 F 0 "R15" V 4380 3400 50  0000 C CNN
 F 1 "0" V 4300 3400 50  0000 C CNN
-F 2 "Resistors_SMD:R_0603" V 4230 3400 50  0001 C CNN
+F 2 "Resistors_SMD:R_0603_HandSoldering" V 4230 3400 50  0001 C CNN
 F 3 "" H 4300 3400 50  0001 C CNN
 	1    4300 3400
@@
 F 0 "R16" V 4580 3400 50  0000 C CNN
 F 1 "0" V 4500 3400 50  0000 C CNN
-F 2 "Resistors_SMD:R_0603" V 4430 3400 50  0001 C CNN
+F 2 "Resistors_SMD:R_0603_HandSoldering" V 4430 3400 50  0001 C CNN
 F 3 "" H 4500 3400 50  0001 C CNN
 	1    4500 3400
@@
 F 0 "R17" V 5130 3400 50  0000 C CNN
 F 1 "10k" V 5050 3400 50  0000 C CNN
-F 2 "Resistors_SMD:R_0603" V 4980 3400 50  0001 C CNN
+F 2 "Resistors_SMD:R_0603_HandSoldering" V 4980 3400 50  0001 C CNN
 F 3 "" H 5050 3400 50  0001 C CNN
 	1    5050 3400
@@
 F 0 "R13" V 6680 3200 50  0000 C CNN
 F 1 "10k" V 6600 3200 50  0000 C CNN
-F 2 "Resistors_SMD:R_0603" V 6530 3200 50  0001 C CNN
+F 2 "Resistors_SMD:R_0603_HandSoldering" V 6530 3200 50  0001 C CNN
 F 3 "" H 6600 3200 50  0001 C CNN
 	1    6600 3200
@@
 Connection ~ 6600 3350
 $Comp
-L +3.3V #PWR28
+L +3.3V #PWR033
 U 1 1 599D7C09
 P 6600 3050
-F 0 "#PWR28" H 6600 2900 50  0001 C CNN
+F 0 "#PWR033" H 6600 2900 50  0001 C CNN
 F 1 "+3.3V" H 6600 3190 50  0000 C CNN
 F 2 "" H 6600 3050 50  0001 C CNN

Commit message: First released
Connections:
- net +3.3VA is gone; now on net +3V3: U2.1 (VIN), U2.3 (EN)
Changed lines of the file:
@@
-	1    0    0    -1
-$EndComp
-$Comp
-L +3.3VA #PWR029
-U 1 1 599B07B0
-P 8250 2050
-F 0 "#PWR029" H 8250 1900 50  0001 C CNN
-F 1 "+3.3VA" H 8250 2190 50  0000 C CNN
-F 2 "" H 8250 2050 50  0001 C CNN
-F 3 "" H 8250 2050 50  0001 C CNN
-	1    8250 2050
 	1    0    0    -1
 $EndComp
@@
 	1    0    0    -1
 $EndComp
+$Comp
+L +3.3V #PWR?
+U 1 1 5AE1B2B7
+P 8250 2050
+F 0 "#PWR?" H 8250 1900 50  0001 C CNN
+F 1 "+3.3V" H 8250 2190 50  0000 C CNN
+F 2 "" H 8250 2050 50  0001 C CNN
+F 3 "" H 8250 2050 50  0001 C CNN
+	1    8250 2050
+	1    0    0    -1
+$EndComp
